File: schematics/kicad/MainScheme.kicad_sch (KiCad schematic)
At the start: 11 parts, among them J1 Raspberry Pi 4, U1 L298N

Commit message: update schematics
Connections:
- net LB Encoder is gone; now on net RA Encoder: A2.20 (A1)
- net Battery Level: now also A2.19 (A0); no longer A2.25 (A6)
- net LA Encoder: now also A2.13 (D10); no longer A2.19 (A0)
- net RA Encoder: no longer A2.21 (A2)
- net RB Encoder: now also A2.21 (A2); no longer A2.22 (A3)
- net TX RP2040: now reaches J1.27 (ID_SD/GPIO0)
- net RX RP2040: now reaches J1.28 (ID_SC/GPIO1)
- net SCL RP2040: no longer names the net of J1.5 (SCL/GPIO3)
- net SCL Rpi: no longer names the net of A2.24 (SCL/A5)
- net SDA RP2040: no longer names the net of J1.3 (SDA/GPIO2)
- net SDA Rpi: no longer names the net of A2.23 (SDA/A4)
